File: Livolo_EU_1Gang_1way.kicad_pcb (KiCad board)
At the start: 2 copper layers, 43 x 43 mm, 31 parts, among them IC1 ATMEGA328P, U1 ATSHA204A, U2 NRF24L01, U3 MTCH102, U6 Touch

Commit message: move MTSA pin to a PWM pin of the ATMEGA
Connections:
- IC1 pad 10: /LED1 -> /MTSA
- IC1 pad 11: /MTPM -> /LED1
- IC1 pad 28: /MTSA -> (no net)
- U3 pad 4: /MTPM -> VCC
Routing:
- net /MTPM: track 18.0 -> 0.00 mm, vias 2 -> 0
- net /MTSA: track 4.06 -> 14.3 mm, vias 0 -> 2
- net VCC: track 115.0 -> 118.6 mm
Other:
- board text added: "v1.1beta - Tonnerre33 27/08/2017"
- board text removed: "v1.0beta - Tonnerre33 05/08/2017"

Commit message: remove resistor for guard
Parts:
- removed R9: 0*, Resistors_SMD:R_0603
Connections:
- U3 pad 6: Net-(R9-Pad1) -> GND
Routing:
- net Net-(R9-Pad1): track 2.48 -> 0.00 mm, vias 1 -> 0
- net GND: track 152.9 -> 151.4 mm, vias 11 -> 10
Changed lines of the file:
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@@
 (kicad_pcb (version 4) (host pcbnew 4.0.6)
   (general
-    (links 73)
+    (links 72)
     (no_connects 0)
     (area 126.926099 83.428599 170.076101 126.578601)
     (thickness 1.6)
     (drawings 31)
-    (tracks 401)
+    (tracks 392)
     (zones 0)
-    (modules 31)
-    (nets 28)
+    (modules 30)
+    (nets 27)
   )
   (page A4)
@@
   (net 25 "Net-(R14-Pad2)")
   (net 26 "Net-(R15-Pad2)")
-  (net 27 "Net-(R9-Pad1)")
   (net_class Default "Ceci est la Netclass par défaut"
     (clearance 0.254)
@@
     (add_net "Net-(R15-Pad1)")
     (add_net "Net-(R15-Pad2)")
-    (add_net "Net-(R9-Pad1)")
   )
   (net_class Power ""
@@
       (net 20 "Net-(C4-Pad1)"))
     (pad 6 smd rect (at 2.2 -0.325) (size 1.45 0.45) (layers Bottom B.Paste B.Mask)
-      (net 27 "Net-(R9-Pad1)"))
+      (net 1 GND))
     (pad 7 smd rect (at 2.2 0.325) (size 1.45 0.45) (layers Bottom B.Paste B.Mask)
       (net 17 /TOUCH_L))
@@
     )
   )
-  (module Resistors_SMD:R_0603 (layer Top)
-    (at 167.894 114.0032 270)
-    (descr "Resistor SMD 0603, reflow soldering, Vishay (see dcrcw.pdf)")
-    (tags "resistor 0603")
-    (attr smd)
-    (fp_text reference R9 (at 0 -1.45 270) (layer F.SilkS)
-      (effects (font (size 1 1) (thickness 0.15)))
-    )
-    (fp_text value 0* (at 0 1.5 270) (layer F.Fab)
-      (effects (font (size 1 1) (thickness 0.15)))
-    )
-    (fp_text user %R (at 0 0 270) (layer F.Fab)
-      (effects (font (size 0.4 0.4) (thickness 0.075)))
-    )
-    (fp_line (start -0.8 0.4) (end -0.8 -0.4) (layer F.Fab) (width 0.1))
-    (fp_line (start 0.8 0.4) (end -0.8 0.4) (layer F.Fab) (width 0.1))
-    (fp_line (start 0.8 -0.4) (end 0.8 0.4) (layer F.Fab) (width 0.1))
-    (fp_line (start -0.8 -0.4) (end 0.8 -0.4) (layer F.Fab) (width 0.1))
-    (fp_line (start 0.5 0.68) (end -0.5 0.68) (layer F.SilkS) (width 0.12))
-    (fp_line (start -0.5 -0.68) (end 0.5 -0.68) (layer F.SilkS) (width 0.12))
-    (fp_line (start -1.25 -0.7) (end 1.25 -0.7) (layer F.CrtYd) (width 0.05))
-    (fp_line (start -1.25 -0.7) (end -1.25 0.7) (layer F.CrtYd) (width 0.05))
-    (fp_line (start 1.25 0.7) (end 1.25 -0.7) (layer F.CrtYd) (width 0.05))
-    (fp_line (start 1.25 0.7) (end -1.25 0.7) (layer F.CrtYd) (width 0.05))
-    (pad 1 smd rect (at -0.75 0 270) (size 0.5 0.9) (layers Top F.Paste F.Mask)
-      (net 27 "Net-(R9-Pad1)"))
-    (pad 2 smd rect (at 0.75 0 270) (size 0.5 0.9) (layers Top F.Paste F.Mask)
-      (net 1 GND))
-    (model ${KISYS3DMOD}/Resistors_SMD.3dshapes/R_0603.wrl
-      (at (xyz 0 0 0))
-      (scale (xyz 1 1 1))
-      (rotate (xyz 0 0 0))
-    )
-  )
   (gr_text VER:C0 (at 134.2644 106.8912) (layer F.SilkS)
     (effects (font (size 0.9652 0.9652) (thickness 0.08128)) (justify bottom))
@@
     (effects (font (size 0.77216 0.77216) (thickness 0.065024)) (justify bottom))
   )
+  (segment (start 165.6236 113.3226) (end 164.1856 113.3226) (width 0.3048) (layer Bottom) (net 1))
   (segment (start 161.8742 101.227) (end 161.8742 101.7858) (width 0.3048) (layer Top) (net 1))
   (segment (start 154.5844 116.6956) (end 154.4828 116.6956) (width 0.3048) (layer Top) (net 1))
@@
   (segment (start 162.9664 111.7172) (end 160.8988 111.7172) (width 0.3048) (layer Bottom) (net 1))
   (segment (start 164.1856 112.9364) (end 162.9664 111.7172) (width 0.3048) (layer Bottom) (net 1))
-  (segment (start 164.1856 114.4096) (end 164.1856 112.9364) (width 0.3048) (layer Bottom) (net 1))
+  (segment (start 164.1856 114.4096) (end 164.1856 113.3226) (width 0.3048) (layer Bottom) (net 1))
+  (segment (start 164.1856 113.3226) (end 164.1856 112.9364) (width 0.3048) (layer Bottom) (net 1))
   (segment (start 164.3986 114.6226) (end 164.1856 114.4096) (width 0.3048) (layer Bottom) (net 1))
   (segment (start 149.4712 115.07) (end 149.4712 116.256) (width 0.3048) (layer Bottom) (net 1) (status 10))
@@
   (segment (start 152.8064 118.1688) (end 152.9588 118.3212) (width 0.3048) (layer Bottom) (net 1))
   (via (at 152.9588 118.3212) (size 0.8128) (drill 0.4064) (layers Top Bottom) (net 1))
-  (segment (start 165.6236 114.6226) (end 166.4814 114.6226) (width 0.3048) (layer Bottom) (net 1) (status 10))
-  (segment (start 167.2456 114.7532) (end 167.894 114.7532) (width 0.3048) (layer Top) (net 1) (status 20))
-  (segment (start 166.9288 115.07) (end 167.2456 114.7532) (width 0.3048) (layer Top) (net 1))
-  (via (at 166.9288 115.07) (size 0.8128) (drill 0.4064) (layers Top Bottom) (net 1))
-  (segment (start 166.4814 114.6226) (end 166.9288 115.07) (width 0.3048) (layer Bottom) (net 1))
-  (segment (start 167.5504 114.7532) (end 167.894 114.7532) (width 0.254) (layer Top) (net 1) (status 30))
   (segment (start 164.4244 116.34) (end 164.4244 117.6252) (width 0.254) (layer Bottom) (net 1) (status 10))
   (segment (start 164.4244 117.6252) (end 164.084 117.9656) (width 0.254) (layer Bottom) (net 1))
@@
   (segment (start 153.7716 91.3464) (end 152.2476 92.8704) (width 0.3048) (layer Bottom) (net 1))
   (via (at 152.2476 92.8704) (size 0.8128) (drill 0.4064) (layers Top Bottom) (net 1))
-  (segment (start 161.2236 112.6726) (end 162.3978 112.6726) (width 0.254) (layer Bottom) (net 2) (status 10))
-  (segment (start 163.322 113.5968) (end 163.322 114.6636) (width 0.254) (layer Bottom) (net 2))
-  (segment (start 162.3978 112.6726) (end 163.322 113.5968) (width 0.254) (layer Bottom) (net 2))
+  (segment (start 162.5244 116.34) (end 162.5244 115.9234) (width 0.254) (layer Bottom) (net 2) (status 10))
+  (segment (start 162.5244 115.9234) (end 161.2236 114.6226) (width 0.3048) (layer Bottom) (net 2) (status 20))
+  (segment (start 161.2236 112.6726) (end 162.3978 112.6726) (width 0.3048) (layer Bottom) (net 2) (status 10))
+  (segment (start 162.3978 112.6726) (end 163.322 113.5968) (width 0.3048) (layer Bottom) (net 2))
+  (segment (start 163.322 113.5968) (end 163.322 114.6636) (width 0.3048) (layer Bottom) (net 2))
   (segment (start 156.8704 86.9624) (end 158.06424 86.9624) (width 0.3048) (layer Bottom) (net 2) (status 30))
   (segment (start 158.06424 86.9624) (end 158.51378 87.41194) (width 0.3048) (layer Bottom) (net 2) (status 30))
@@
   (segment (start 164.20338 99.35502) (end 164.20338 109.482) (width 0.3048) (layer Top) (net 2))
   (segment (start 164.20338 109.482) (end 164.20338 113.78222) (width 0.3048) (layer Top) (net 2))
+  (segment (start 164.20338 113.78222) (end 163.322 114.6636) (width 0.3048) (layer Top) (net 2))
+  (via (at 163.322 114.6636) (size 0.8128) (drill 0.4064) (layers Top Bottom) (net 2))
   (segment (start 162.5244 115.4612) (end 162.5244 116.34) (width 0.3048) (layer Bottom) (net 2) (status 20))
   (segment (start 163.322 114.6636) (end 162.5244 115.4612) (width 0.3048) (layer Bottom) (net 2))
-  (via (at 163.322 114.6636) (size 0.8128) (drill 0.4064) (layers Top Bottom) (net 2))
-  (segment (start 164.20338 113.78222) (end 163.322 114.6636) (width 0.3048) (layer Top) (net 2))
   (via (at 164.20338 99.35502) (size 0.8128) (drill 0.4064) (layers Top Bottom) (net 2))
   (segment (start 164.3888 95.6136) (end 163.322 94.5468) (width 0.3048) (layer Top) (net 2))
@@
   (segment (start 138.9888 117.2036) (end 146.7612 117.2036) (width 0.3048) (layer Bottom) (net 2))
   (segment (start 136.4742 120.2184) (end 136.4742 119.8706) (width 0.3048) (layer Bottom) (net 2) (status 30))
-  (segment (start 162.5244 116.34) (end 162.5244 115.9234) (width 0.254) (layer Bottom) (net 2) (status 10))
-  (segment (start 162.5244 115.9234) (end 161.2236 114.6226) (width 0.254) (layer Bottom) (net 2) (status 20))
   (segment (start 162.4252 108.2628) (end 162.4252 107.4832) (width 0.254) (layer Bottom) (net 3) (status 10))
   (segment (start 163.22802 106.68038) (end 163.22802 105.64406) (width 0.254) (layer Bottom) (net 3) (status 20))
@@
   (segment (start 157.734 112.8856) (end 149.9362 105.0878) (width 0.254) (layer Bottom) (net 26) (status 20))
   (segment (start 149.9362 105.0878) (end 148.4884 105.0878) (width 0.254) (layer Bottom) (net 26) (status 30))
-  (segment (start 167.894 113.2532) (end 167.2456 113.2532) (width 0.254) (layer Top) (net 27) (status 10))
-  (segment (start 166.7458 113.3226) (end 165.6236 113.3226) (width 0.254) (layer Bottom) (net 27) (status 20))
-  (segment (start 167.0304 113.038) (end 166.7458 113.3226) (width 0.254) (layer Bottom) (net 27))
-  (via (at 167.0304 113.038) (size 0.6858) (drill 0.3302) (layers Top Bottom) (net 27))
-  (segment (start 167.2456 113.2532) (end 167.0304 113.038) (width 0.254) (layer Top) (net 27))
   (zone (net 1) (net_name GND) (layer Bottom) (hatch edge 0.508)
     (connect_pads (clearance 0.381))
