File: Livolo_EU_1Gang_1way.sch (KiCad schematic (older format))
At the start: 31 parts, among them IC1 ATMEGA328P, U1 ATSHA204A, U2 NRF24L01, U3 MTCH102, U6 Touch

Commit message: move MTSA pin to a PWM pin of the ATMEGA
Connections:
- net LED1: now also IC1.11 (PD7(AIN1)); no longer IC1.10 (PD6(AIN0))
- net MTSA: now also IC1.10 (PD6(AIN0)); no longer IC1.28 (PC5(ADC5/SCL))
- net VCC: now also U3.4 (MTPM)
- removed net MTPM: IC1.11 (PD7(AIN1)), U3.4 (MTPM)
- no-connect marks 24 -> 25
Changed lines of the file:
@@
 LIBS:touch
 LIBS:MTCH102
-LIBS:Livolo_EU_1Gang_1way-cache
 EELAYER 25 0
 EELAYER END
@@
 Sheet 1 1
 Title "Linovo_EU_1Gang_1way.sch"
-Date "2017-08-05"
-Rev "v1.0beta"
+Date "2017-08-27"
+Rev "v1.1beta"
 Comp ""
 Comment1 "VL-C701X-2 VER C0"
@@
 Text Label 8950 4650 2    65   ~ 0
 CSN
-Text Label 8950 4150 2    65   ~ 0
+Text Label 8950 4250 2    65   ~ 0
 LED1
 Text Label 8950 3750 2    65   ~ 0
@@
 	-1   0    0    1
 $EndComp
-Text Label 8950 4250 2    65   ~ 0
-MTPM
 $Comp
 L LED D2
@@
 Text Label 15650 2800 2    65   ~ 0
 MTSA
-Text Label 12900 2800 2    65   ~ 0
-MTPM
 $Comp
 L Touch U6
@@
 	12900 2500 13000 2500
 Wire Wire Line
-	12950 2350 12950 2500
+	12950 2350 12950 2800
 Connection ~ 12950 2500
 Connection ~ 15050 2800
@@
 Wire Wire Line
 	8450 4050 8950 4050
-Text Label 8950 3150 2    65   ~ 0
+Text Label 8950 4150 2    65   ~ 0
 MTSA
-Wire Wire Line
-	8950 3150 8450 3150
 NoConn ~ 8450 3250
-Wire Wire Line
-	8950 4250 8450 4250
 NoConn ~ 10950 8750
 Wire Wire Line
@@
 	12500 2700 13000 2700
 Wire Wire Line
-	13000 2800 12900 2800
-Wire Wire Line
 	14500 2700 14600 2700
+Wire Wire Line
+	12950 2800 13000 2800
+Wire Wire Line
+	8950 4250 8450 4250
+NoConn ~ 8450 3150
 $EndSCHEMATC

Commit message: remove resistor for guard
Parts:
- removed R9: 0*, Resistors_SMD:R_0603, symbol R_Small
Connections:
- net GND: now also U3.6 (MTO1/GC)
Changed lines of the file:
@@
 LIBS:touch
 LIBS:MTCH102
+LIBS:Livolo_EU_1Gang_1way-cache
 EELAYER 25 0
 EELAYER END
@@
 Wire Wire Line
 	14500 2800 15150 2800
-$Comp
-L R_Small R9
-U 1 1 597CCC76
-P 14700 2700
-F 0 "R9" H 14730 2720 50  0000 L CNN
-F 1 "0*" H 14730 2660 50  0000 L CNN
-F 2 "Resistors_SMD:R_0603" H 14700 2700 50  0001 C CNN
-F 3 "" H 14700 2700 50  0001 C CNN
-	1    14700 2700
-	0    -1   -1   0
-$EndComp
 Wire Wire Line
 	10950 8150 10850 8150
@@
 	12500 2700 13000 2700
 Wire Wire Line
-	14500 2700 14600 2700
-Wire Wire Line
 	12950 2800 13000 2800
 Wire Wire Line
 	8950 4250 8450 4250
 NoConn ~ 8450 3150
+Wire Wire Line
+	14800 2700 14500 2700
 $EndSCHEMATC
